File: sid-board-kicad/sid-board-v3.kicad_pcb (KiCad board)
At the start: 2 copper layers, 60.1 x 60.1 mm, 49 parts, among them J1 SPI + UART, J2 ESP32 UART, J3 Conn_01x08, Q1 BSS138, SW1 EN, SW2 FLASH, U1 SC16IS752, U2 MCP1703A-3302, U3 SN65HVD232 x3, U4 SN65HVD232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

Commit message: More labelling
Parts:
- J1: value SPI + UART -> SPI
- J2: value ESP32 UART -> UART
Other:
- board text added: "+"
- board text added: "-"
- board text added: "3.3V"
- board text added: "CL"
- board text added: "CS"
- board text added: "GND"
- board text added: "H"
- board text added: "I-BUS"
- board text added: "ICM"
- board text added: "IO22 (DIN)"
- board text added: "IO25 (WSEL)"
- board text added: "IO27"
- board text added: "IO27 (BCLK)"
- board text added: "IO32"
- board text added: "IO33"
- board text added: "L"
- board text added: "S0"
- board text added: "SI"
- board text added: "SID"
Changed lines of the file:
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@@
   (general
     (thickness 1.6)
-    (drawings 12)
+    (drawings 82)
     (tracks 1757)
     (zones 0)
@@
     (0 F.Cu signal)
     (31 B.Cu signal)
-    (32 B.Adhes user)
-    (33 F.Adhes user)
-    (34 B.Paste user)
+    (32 B.Adhes user hide)
+    (33 F.Adhes user hide)
+    (34 B.Paste user hide)
     (35 F.Paste user)
-    (36 B.SilkS user)
+    (36 B.SilkS user hide)
     (37 F.SilkS user)
-    (38 B.Mask user)
+    (38 B.Mask user hide)
     (39 F.Mask user)
-    (40 Dwgs.User user)
-    (41 Cmts.User user)
-    (42 Eco1.User user)
-    (43 Eco2.User user)
+    (40 Dwgs.User user hide)
+    (41 Cmts.User user hide)
+    (42 Eco1.User user hide)
+    (43 Eco2.User user hide)
     (44 Edge.Cuts user)
-    (45 Margin user)
-    (46 B.CrtYd user)
+    (45 Margin user hide)
+    (46 B.CrtYd user hide)
     (47 F.CrtYd user)
-    (48 B.Fab user)
+    (48 B.Fab user hide)
     (49 F.Fab user)
   )
@@
       (effects (font (size 1 1) (thickness 0.15)))
     )
-    (fp_text value "SPI + UART" (at 4.445 4.318 90) (layer F.SilkS)
+    (fp_text value SPI (at 1.016 -2.159 180) (layer F.SilkS)
       (effects (font (size 1 1) (thickness 0.15)))
     )
@@
       (effects (font (size 1 1) (thickness 0.15)))
     )
-    (fp_text value "ESP32 UART" (at 0 -3.556 90) (layer F.SilkS)
+    (fp_text value UART (at -5.334 0.254 180) (layer F.SilkS)
       (effects (font (size 1 1) (thickness 0.15)))
     )
@@
     )
   )
+  (gr_text CS (at 167.005 85.09 90) (layer F.SilkS)
+    (effects (font (size 0.6 0.6) (thickness 0.15)))
+  )
+  (gr_text SI (at 165.735 85.09 90) (layer F.SilkS)
+    (effects (font (size 0.6 0.6) (thickness 0.15)))
+  )
+  (gr_text CL (at 165.735 83.82 90) (layer F.SilkS)
+    (effects (font (size 0.6 0.6) (thickness 0.15)))
+  )
+  (gr_text "S0\n" (at 167.005 83.82 90) (layer F.SilkS)
+    (effects (font (size 0.6 0.6) (thickness 0.15)))
+  )
+  (gr_text + (at 167.005 80.01) (layer F.SilkS)
+    (effects (font (size 0.7 0.7) (thickness 0.15)))
+  )
+  (gr_text + (at 167.005 81.28) (layer F.SilkS)
+    (effects (font (size 0.7 0.7) (thickness 0.15)))
+  )
+  (gr_text + (at 167.005 82.55) (layer F.SilkS)
+    (effects (font (size 0.7 0.7) (thickness 0.15)))
+  )
+  (gr_text - (at 165.735 82.55) (layer F.SilkS)
+    (effects (font (size 0.7 0.7) (thickness 0.15)))
+  )
+  (gr_text - (at 165.735 81.28) (layer F.SilkS)
+    (effects (font (size 0.7 0.7) (thickness 0.15)))
+  )
+  (gr_text - (at 165.735 80.01) (layer F.SilkS)
+    (effects (font (size 0.7 0.7) (thickness 0.15)))
+  )
+  (gr_line (start 165.1 79.375) (end 166.37 79.375) (layer F.SilkS) (width 0.15))
+  (gr_line (start 165.1 80.645) (end 165.1 79.375) (layer F.SilkS) (width 0.15))
+  (gr_line (start 167.64 79.375) (end 167.64 80.645) (layer F.SilkS) (width 0.15))
+  (gr_line (start 166.37 79.375) (end 167.64 79.375) (layer F.SilkS) (width 0.15))
+  (gr_line (start 166.37 80.645) (end 166.37 79.375) (layer F.SilkS) (width 0.15))
+  (gr_line (start 167.64 80.645) (end 166.37 80.645) (layer F.SilkS) (width 0.15))
+  (gr_line (start 167.64 81.915) (end 167.64 80.645) (layer F.SilkS) (width 0.15))
+  (gr_line (start 166.37 80.645) (end 166.37 81.915) (layer F.SilkS) (width 0.15))
+  (gr_line (start 165.1 80.645) (end 166.37 80.645) (layer F.SilkS) (width 0.15))
+  (gr_line (start 165.1 81.915) (end 165.1 80.645) (layer F.SilkS) (width 0.15))
+  (gr_line (start 167.64 81.915) (end 166.37 81.915) (layer F.SilkS) (width 0.15))
+  (gr_line (start 167.64 83.185) (end 167.64 81.915) (layer F.SilkS) (width 0.15))
+  (gr_line (start 166.37 81.915) (end 166.37 83.185) (layer F.SilkS) (width 0.15))
+  (gr_line (start 165.1 81.915) (end 166.37 81.915) (layer F.SilkS) (width 0.15))
+  (gr_line (start 165.1 83.185) (end 165.1 81.915) (layer F.SilkS) (width 0.15))
+  (gr_line (start 167.64 83.185) (end 166.37 83.185) (layer F.SilkS) (width 0.15))
+  (gr_line (start 167.64 84.455) (end 167.64 83.185) (layer F.SilkS) (width 0.15))
+  (gr_line (start 166.37 83.185) (end 166.37 84.455) (layer F.SilkS) (width 0.15))
+  (gr_line (start 165.1 83.185) (end 166.37 83.185) (layer F.SilkS) (width 0.15))
+  (gr_line (start 165.1 84.455) (end 165.1 83.185) (layer F.SilkS) (width 0.15))
+  (gr_line (start 167.64 84.455) (end 167.64 85.725) (layer F.SilkS) (width 0.15))
+  (gr_line (start 166.37 84.455) (end 167.64 84.455) (layer F.SilkS) (width 0.15))
+  (gr_line (start 166.37 84.455) (end 166.37 85.725) (layer F.SilkS) (width 0.15))
+  (gr_line (start 165.1 84.455) (end 166.37 84.455) (layer F.SilkS) (width 0.15))
+  (gr_line (start 165.1 85.725) (end 165.1 84.455) (layer F.SilkS) (width 0.15))
+  (gr_line (start 167.64 85.725) (end 165.1 85.725) (layer F.SilkS) (width 0.15))
+  (gr_text H (at 120.65 78.74) (layer F.SilkS)
+    (effects (font (size 0.7 0.7) (thickness 0.15)))
+  )
+  (gr_text L (at 119.38 78.74) (layer F.SilkS)
+    (effects (font (size 0.7 0.7) (thickness 0.15)))
+  )
+  (gr_line (start 121.285 79.375) (end 120.015 79.375) (layer F.SilkS) (width 0.15))
+  (gr_line (start 121.285 78.105) (end 121.285 79.375) (layer F.SilkS) (width 0.15))
+  (gr_line (start 120.015 78.105) (end 121.285 78.105) (layer F.SilkS) (width 0.15))
+  (gr_line (start 120.015 78.105) (end 118.745 78.105) (layer F.SilkS) (width 0.15))
+  (gr_line (start 120.015 79.375) (end 120.015 78.105) (layer F.SilkS) (width 0.15))
+  (gr_line (start 118.745 79.375) (end 120.015 79.375) (layer F.SilkS) (width 0.15))
+  (gr_line (start 118.745 78.105) (end 118.745 79.375) (layer F.SilkS) (width 0.15))
+  (gr_text SID (at 164.846 66.802) (layer F.SilkS)
+    (effects (font (size 1 1) (thickness 0.15)))
+  )
+  (gr_text ICM (at 146.05 66.802) (layer F.SilkS)
+    (effects (font (size 1 1) (thickness 0.15)))
+  )
+  (gr_text I-BUS (at 123.698 66.802) (layer F.SilkS)
+    (effects (font (size 1 1) (thickness 0.15)))
+  )
+  (gr_circle (center 156.972 109.22) (end 157.226 109.22) (layer F.SilkS) (width 0.15))
+  (gr_circle (center 160.401 75.565) (end 160.655 75.565) (layer F.SilkS) (width 0.15))
+  (gr_circle (center 160.401 90.551) (end 160.655 90.551) (layer F.SilkS) (width 0.15))
+  (gr_line (start 126.238 82.042) (end 125.603 81.661) (layer B.SilkS) (width 0.15))
+  (gr_line (start 126.238 81.28) (end 126.238 82.042) (layer B.SilkS) (width 0.15))
+  (gr_line (start 125.603 81.661) (end 126.238 81.28) (layer B.SilkS) (width 0.15))
+  (gr_line (start 125.603 81.026) (end 125.603 82.296) (layer B.SilkS) (width 0.15))
+  (gr_line (start 120.523 84.582) (end 121.158 84.201) (layer B.SilkS) (width 0.15))
+  (gr_line (start 120.523 83.82) (end 120.523 84.582) (layer B.SilkS) (width 0.15))
+  (gr_line (start 121.158 84.201) (end 120.523 83.82) (layer B.SilkS) (width 0.15))
+  (gr_line (start 121.158 83.566) (end 121.158 84.836) (layer B.SilkS) (width 0.15))
+  (gr_circle (center 136.398 85.598) (end 136.652 85.598) (layer B.SilkS) (width 0.15))
+  (gr_circle (center 144.272 85.598) (end 144.526 85.598) (layer B.SilkS) (width 0.15))
+  (gr_circle (center 151.892 85.598) (end 152.146 85.598) (layer B.SilkS) (width 0.15))
+  (gr_text GND (at 129.794 120.142 -90) (layer B.SilkS)
+    (effects (font (size 1 1) (thickness 0.2)) (justify left mirror))
+  )
+  (gr_text 3.3V (at 132.334 120.142 -90) (layer B.SilkS)
+    (effects (font (size 1 1) (thickness 0.2)) (justify left mirror))
+  )
+  (gr_text IO32 (at 134.874 120.142 -90) (layer B.SilkS)
+    (effects (font (size 1 1) (thickness 0.2)) (justify left mirror))
+  )
+  (gr_text IO33 (at 137.414 120.142 -90) (layer B.SilkS)
+    (effects (font (size 1 1) (thickness 0.2)) (justify left mirror))
+  )
+  (gr_text IO27 (at 139.954 120.142 -90) (layer B.SilkS)
+    (effects (font (size 1 1) (thickness 0.2)) (justify left mirror))
+  )
+  (gr_text "IO22 (DIN)" (at 142.494 120.142 -90) (layer B.SilkS)
+    (effects (font (size 1 1) (thickness 0.2)) (justify left mirror))
+  )
+  (gr_text "IO25 (WSEL)" (at 145.034 120.142 -90) (layer B.SilkS)
+    (effects (font (size 1 1) (thickness 0.2)) (justify left mirror))
+  )
+  (gr_text "IO27 (BCLK)" (at 147.574 120.142 -90) (layer B.SilkS)
+    (effects (font (size 1 1) (thickness 0.2)) (justify left mirror))
+  )
   (gr_arc (start 170.316 120.786) (end 170.316 123.328739) (angle -90) (layer Edge.Cuts) (width 0.1))
